Commit message: support hokuyo sesnor

File: ca_description/urdf/create_base.urdf.xacro (robot description, xacro)
@@ -31,4 +31,5 @@
   <xacro:macro name="create_base" params="diffdrive_update_rate:=40 wheel_separation wheel_radius:=0.036 wheel_width:=0.024 wheel_torque:=1.0 wheel_accel:=1.8 mass_kg:=3.5 base_diameter *mesh">
     <xacro:include filename="$(find ca_description)/urdf/create_base_gazebo.urdf.xacro" />
+    <xacro:include filename="$(find ca_description)/urdf/sensors/hokuyo.urdf.xacro" />
     <link name="base_footprint">
     <visual>
@@ -132,4 +133,5 @@
     <xacro:create_wheel prefix="left" y_offset="${wheel_separation / 2}" wheel_radius="${wheel_radius}" wheel_width="${wheel_width}"/>
     <xacro:create_wheel prefix="right" y_offset="${wheel_separation / -2}" wheel_radius="${wheel_radius}" wheel_width="${wheel_width}"/>
+    <xacro:sensor_hokuyo parent="base_link" />
     <!--<link name="rear_wheel_link">
     <inertial>
@@ -202,4 +204,5 @@
     <xacro:sim_create_cliff_sensors/>
     <xacro:sim_imu/>
+    <xacro:sim_create_hokuyo_sensor update_rate="20" min_angle="-130" max_angle="130" ray_count="180"/>
   </xacro:macro>
 </robot>

File: ca_description/urdf/create_base_gazebo.urdf.xacro (robot description, xacro)
@@ -1,4 +1,5 @@
 <?xml version="1.0" ?>
 <robot xmlns:xacro="http://ros.org/wiki/xacro">
+	<xacro:property name="M_PI" value="3.1415926535897931" />
   <xacro:macro name="sim_create_base">
     <gazebo>
@@ -195,3 +196,36 @@
     </gazebo>
   </xacro:macro>
+  <xacro:macro name="sim_create_hokuyo_sensor" params="update_rate min_angle max_angle ray_count">
+  	<gazebo reference="laser_link">
+    	<sensor type="ray" name="laser">
+		    <always_on>true</always_on>
+		    <update_rate>${update_rate}</update_rate>
+		    <pose>0 0 0 0 0 0</pose>
+		    <visualize>false</visualize>
+				<displayRays>false</displayRays>
+		    <ray>
+		      <scan>
+		        <horizontal>
+		          <samples>${ray_count}</samples>
+		          <resolution>1</resolution>
+		          <min_angle>${min_angle * M_PI/180}</min_angle>
+		          <max_angle>${max_angle * M_PI/180}</max_angle>
+		        </horizontal>
+		      </scan>
+          <range>
+		        <min>0.08</min>
+		        <max>30.0</max>
+		        <resolution>0.01</resolution>
+          </range>
+        </ray>
+        <plugin name="gazebo_ros_laser_controller" filename="libgazebo_ros_laser.so">
+		      <gaussianNoise>0.005</gaussianNoise>
+		      <alwaysOn>true</alwaysOn>
+		      <updateRate>${update_rate}</updateRate>
+		      <topicName>scan</topicName>
+		      <frameName>laser_link</frameName>
+        </plugin>
+    	</sensor>
+		</gazebo>
+  </xacro:macro>
 </robot>
